File: epdiy-v7-model-F/epaper-breakout.kicad_sch (KiCad schematic)
At the start: 123 parts, among them J1 USB_C_Receptacle_USB2.0, J2 EXTENSION_HEADER, J3 SM04B-SRSS-TB_LF__SN_, J4 XF2M-3315-1A, J5 CONN_BAT, J6 8BIT_HEADER, J7 ESP_HDR, J8 ED133UT2, J9 USB_C_Receptacle_USB2.0, Q1 AO3401A, Q3 MMBT3904, Q4 MMBT3904, U1 MCP1700-3302E_SOT23, U10 RT9080-33GJ5, U11 TP4056, U2 PCA9535PW, U3 TPS651851RSLR, U4 USBLC6-2P6, U5 XC6206PxxxMR, U6 ED078KH6, U8 ESP32-S3-WROOM-1, U9 CH340C, Y1 RV-3032-C7

Commit message: Starting to accomodate stuff over the board
Parts:
- removed C13, C14, C18: 1uF, Capacitor_SMD:C_0805_2012Metric, symbol Device:C
- removed C19: 10uF, Capacitor_SMD:C_0805_2012Metric, symbol Device:C
- removed C42: 100nF, Capacitor_SMD:C_0805_2012Metric, symbol Device:C
- removed J1: USB_C_Receptacle_USB2.0, Connector_USB:USB_C_Receptacle_HRO_TYPE-C-31-M-12, symbol Connector:USB_C_Receptacle_USB2.0
- removed J2: EXTENSION_HEADER, Connector_PinHeader_2.54mm:PinHeader_1x12_P2.54mm_Vertical, symbol Connector:Conn_01x12_Socket
- removed J7: ESP_HDR, Connector_PinHeader_2.54mm:PinHeader_1x08_P2.54mm_Vertical, symbol Connector:Conn_01x08_Socket
- removed J8: ED133UT2, epaper-breakout:HRS_FH26W-39S-0.3SHW(60), symbol ed133ut2_connector-rescue:ED133UT2-epd_breakout
- removed JP1: VBAT_GPIO2, Jumper:SolderJumper-2_P1.3mm_Bridged2Bar_Pad1.0x1.5mm, symbol Jumper:Jumper_2_Bridged
- removed JP2: RTCINT_GPIO2, Jumper:SolderJumper-2_P1.3mm_Bridged2Bar_Pad1.0x1.5mm, symbol Jumper:Jumper_2_Bridged
- removed Q3, Q4: MMBT3904, Package_TO_SOT_SMD:SOT-23, symbol Transistor_BJT:MMBT3904
- removed R1, R11: 10k, Resistor_SMD:R_0603_1608Metric, symbol Device:R
- removed R2, R7: 5.1k, Resistor_SMD:R_0603_1608Metric, symbol Device:R
- removed U4: USBLC6-2P6, Package_TO_SOT_SMD:SOT-666, symbol Power_Protection:USBLC6-2P6
- removed U5: XC6206PxxxMR, Package_TO_SOT_SMD:SOT-23-3, symbol Regulator_Linear:XC6206PxxxMR
- removed U9: CH340C, Package_SO:SOIC-16_3.9x9.9mm_P1.27mm, symbol Interface_USB:CH340C
- U6: footprint footprints:FH1240S05SH55 -> epaper-breakout:Hirose_FH12-40S-0.5SH_mirrored
Connections:
- net GPIO_2 is gone; now on net ~{GPIO_INTR}: U8.38 (GPIO2/TOUCH2/ADC1_CH1)
- net RTC_INT is gone; now on net GPIO_3: R32.1, Y1.3 (~{INT})
- net CKV: now also U8.35 (MTMS/GPIO42); no longer U8.25 (GPIO48/SPICLK_N/SUBSPICLK_N_DIFF)
- net D0: now also U8.24 (GPIO47/SPICLK_P/SUBSPICLK_P_DIFF); no longer U8.5 (GPIO5/TOUCH5/ADC1_CH4)
- net D1: now also U8.23 (GPIO21); no longer U8.6 (GPIO6/TOUCH6/ADC1_CH5)
- net D10: now also U8.10 (GPIO17/U1TXD/ADC2_CH6); no longer U8.19 (GPIO11/TOUCH11/ADC2_CH0/FSPID/FSPIIO5/SUBSPID)
- net D11: now also U8.9 (GPIO16/U0CTS/ADC2_CH5/XTAL_32K_NH5); no longer U8.20 (GPIO12/TOUCH12/ADC2_CH1/FSPICLK/FSPIIO6/SUBSPICLK)
- net D12: now also U8.8 (GPIO15/U0RTS/ADC2_CH4/XTAL_32K_P); no longer U8.21 (GPIO13/TOUCH13/ADC2_CH2/FSPIQ/FSPIIO7/SUBSPIQ)
- net D13: now also U8.7 (GPIO7/TOUCH7/ADC1_CH6); no longer U8.22 (GPIO14/TOUCH14/ADC2_CH3/FSPIWP/FSPIDQS/SUBSPIWP)
- net D14: now also U8.6 (GPIO6/TOUCH6/ADC1_CH5); no longer U8.23 (GPIO21)
- net D15: now also U8.5 (GPIO5/TOUCH5/ADC1_CH4); no longer U8.24 (GPIO47/SPICLK_P/SUBSPICLK_P_DIFF)
- net D2: now also U8.22 (GPIO14/TOUCH14/ADC2_CH3/FSPIWP/FSPIDQS/SUBSPIWP); no longer U8.7 (GPIO7/TOUCH7/ADC1_CH6)
- net D3: now also U8.21 (GPIO13/TOUCH13/ADC2_CH2/FSPIQ/FSPIIO7/SUBSPIQ); no longer U8.8 (GPIO15/U0RTS/ADC2_CH4/XTAL_32K_P)
- net D4: now also U8.20 (GPIO12/TOUCH12/ADC2_CH1/FSPICLK/FSPIIO6/SUBSPICLK); no longer U8.9 (GPIO16/U0CTS/ADC2_CH5/XTAL_32K_NH5)
- net D5: now also U8.19 (GPIO11/TOUCH11/ADC2_CH0/FSPID/FSPIIO5/SUBSPID); no longer U8.10 (GPIO17/U1TXD/ADC2_CH6)
- net D6: now also U8.18 (GPIO10/TOUCH10/ADC1_CH9/FSPICS0/FSPIIO4/SUBSPICS0); no longer U8.11 (GPIO18/U1RXD/ADC2_CH7/CLK_OUT3)
- net D7: now also U8.17 (GPIO9/TOUCH9/ADC1_CH8/FSPIHD/SUBSPIHD); no longer U8.12 (GPIO8/TOUCH8/ADC1_CH7/SUBSPICS1)
- net D8: now also U8.12 (GPIO8/TOUCH8/ADC1_CH7/SUBSPICS1); no longer U8.17 (GPIO9/TOUCH9/ADC1_CH8/FSPIHD/SUBSPIHD)
- net D9: now also U8.11 (GPIO18/U1RXD/ADC2_CH7/CLK_OUT3); no longer U8.18 (GPIO10/TOUCH10/ADC1_CH9/FSPICS0/FSPIIO4/SUBSPICS0)
- net EP_STV: now also U8.34 (MTDI/GPIO41/CLK_OUT1); no longer U8.26 (GPIO45)
- net GPIO_1: now also C23.2, R21.2, R22.1
- net LEH: now also U8.25 (GPIO48/SPICLK_N/SUBSPICLK_N_DIFF); no longer U8.35 (MTMS/GPIO42)
- net XSTL: now also U8.26 (GPIO45); no longer U8.34 (MTDI/GPIO41/CLK_OUT1)
- net ~{GPIO_INTR}: no longer U8.31 (GPIO38/FSPIWP/SUBSPIWP)
- net EXT1: no longer names the net of U2.4 (IO0_0)
- net EXT2: no longer names the net of U2.5 (IO0_1)
- net EXT3: no longer names the net of U2.6 (IO0_2)
- net EXT4: no longer names the net of U2.7 (IO0_3)
- net EXT5: no longer names the net of U2.8 (IO0_4)
- net EXT6: no longer names the net of U2.9 (IO0_5)
- net EXT7: no longer names the net of U2.10 (IO0_6)
- net EXT8: no longer names the net of U2.11 (IO0_7)
- new net GPIO_38: U8.31 (GPIO38/FSPIWP/SUBSPIWP)
- no-connect marks 19 -> 20
Other:
- note removed: "Auto-Reset"
- note removed: "Button for RESET"
- note removed: "EPD Connector 39pin, 8bit"
- note removed: "ESP Header"
- note removed: "USB Connector"
- note removed: "USB to UART"
- moved on the sheet: C17

Commit message: DRC validation missing
Parts:
- removed TP1: +22V, TestPoint:TestPoint_Pad_D2.5mm, symbol Connector:TestPoint
- removed TP3: -20V, TestPoint:TestPoint_Pad_D2.5mm, symbol Connector:TestPoint
- added U4: TSOP341xx, OptoDevice:Vishay_MOLD-3Pin, symbol Interface_Optical:TSOP341xx
- J6: footprint Connector_PinHeader_2.54mm:PinHeader_1x10_P2.54mm_Vertical -> Connector_PinHeader_2.54mm:PinHeader_1x11_P2.54mm_Vertical; symbol Connector:Conn_01x10_Female -> Connector:Conn_01x11_Socket; now in the parts list
- R22: value 150k -> 680k; LCSC C22807 -> C25822
- TP6: footprint TestPoint:TestPoint_Pad_D1.5mm -> TestPoint:TestPoint_Pad_1.0x1.0mm
Connections:
- net D10: now also J6.4 (Pin_4); no longer J6.3 (Pin_3)
- net D11: now also J6.5 (Pin_5); no longer J6.4 (Pin_4)
- net D12: now also J6.6 (Pin_6); no longer J6.5 (Pin_5)
- net D13: now also J6.7 (Pin_7); no longer J6.6 (Pin_6)
- net D14: now also J6.8 (Pin_8); no longer J6.7 (Pin_7)
- net D15: now also J6.9 (Pin_9); no longer J6.8 (Pin_8)
- net D8: now also J6.2 (Pin_2); no longer J6.1 (Pin_1)
- net D9: now also J6.3 (Pin_3); no longer J6.2 (Pin_2)
- net EPD_VDD: now also J6.10 (Pin_10); no longer J6.9 (Pin_9)
- net GND: now also J6.11 (Pin_11), U4.2 (GND); no longer J6.10 (Pin_10)
- net 3.3V renamed +3V3
- net +3V3: now also U4.3 (Vs)
- net BORDER: no longer names the net of J4.33 (BORDER)
- net BORDER: no longer U6.40 (BORDER)
- net QWIIC_3V3 renamed +3V3_QW
- net USB_RXD renamed IR_OUT
- net IR_OUT: now also U4.1 (OUT)
- net USB_TXD renamed GPIO_44
- net GPIO_44: now also J6.1 (Pin_1)
- no-connect marks 20 -> 21
Other:
- note added: "Breakout Header for unused pins in 8bit mode + extra IO44"
- note added: "IR RECEIVER"
- note removed: "Breakout Header for unused pins in 8bit mode"
- moved on the sheet: C40, J3, R10, R15, R4, R6, Y1

Commit message: First model routed
Parts:
- added C42: 22pF, Capacitor_SMD:C_0402_1005Metric, symbol Device:C
- added SW2, SW3: HX-3X6X3.5-CA-0.6-2.5N, footprint_common:C2686860_button_TC073B-H055-L1, symbol easyeda:HX-3X6X3.5-CA-0.6-2.5N
Connections:
- net EN: now also SW3.2
- net GND: now also C42.1, SW2.1, SW3.1
- net IO0: now also C42.2, SW2.2
- no-connect marks 21 -> 23
Other:
- note added: "IO0 BOOT / USR + RESET"

Commit message: Update 33 pin w/34 and add 2nd USBC
Parts:
- added J10: USB_C_Receptacle_USB2.0, Connector_USB:USB_C_Receptacle_HRO_TYPE-C-31-M-12, symbol Connector:USB_C_Receptacle_USB2.0
- added U12: ED060XC5, footprint_common:X05A20H34G, symbol epd_breakout:ED060XC5
- J4: now not fitted; now left out of the parts list
Connections:
- net +22V: now also U12.34 (VGG)
- net -15V: now also U12.1 (VNEG)
- net -20V: now also U12.2 (VEE)
- net 15V: now also U12.33 (VPOS)
- net CKV: now also U12.28 (CKV)
- net D0: now also U12.13 (D0)
- net D1: now also U12.14 (D1)
- net D2: now also U12.15 (D2)
- net D3: now also U12.16 (D3)
- net D4: now also U12.17 (D4)
- net D5: now also U12.18 (D5)
- net D6: now also U12.19 (D6)
- net D7: now also U12.20 (D7)
- net EPD_VDD: now also U12.6 (VDD)
- net EP_MODE: now also U12.27 (MODE1)
- net EP_OE: now also U12.11 (XOE)
- net EP_STV: now also U12.29 (SPV)
- net EP_VCOM: now also U12.21 (VCOM)
- net ESP_USB+: now also J10.A6 (D+), J10.B6 (D+)
- net ESP_USB-: now also J10.A7 (D-), J10.B7 (D-)
- net GND: now also J10.A1 (GND), J10.A12 (GND), J10.B1 (GND), J10.B12 (GND), J10.S1 (SHIELD), U12.26 (VSS), U12.3 (VSS), U12.32 (VSS), U12.7 (VSS), U12.9 (VSS)
- net LEH: now also U12.10 (XLE)
- net VBUS: now also J10.A4 (VBUS), J10.A9 (VBUS), J10.B4 (VBUS), J10.B9 (VBUS)
- net XCL: now also U12.8 (XCL)
- net XSTL: now also U12.12 (XSTL)
- no-connect marks 23 -> 28
Other:
- note added: "EPD Connector 34pin, 8bit"
- note added: "USB-C LEFT / CDC Serial to MCU"
- note added: "USB-C RIGHT / CDC Serial to MCU"
- note removed: "USB-C JTAG / CDC Serial to MCU"
- moved on the sheet: J9, R12, R13
